File: OpenASCHat/OpenASCHat.sch (KiCad schematic (older format))
At the start: 46 parts, among them J3 40HAT, J6 CONN_02X02, J9 CONN_01X02, Q1 DMG2305UX, Q2 DMMT5401, U2 CAT24C32

Commit message: Some changes
Parts:
- removed Q? (x2): BS107, Package_TO_SOT_THT:TO-92_Inline, symbol Transistor_FET:BS107
- removed Q? (x2): Q_PNP_CEB, symbol Device:Q_PNP_CEB
- removed U?: 74LVC1GU04DRL, Package_TO_SOT_SMD:SOT-553, symbol 74xGxx:74LVC1GU04DRL
- added C?: 1n5, symbol Device:C_Small
- added Q? (x2): BCX51, Package_TO_SOT_SMD:SOT-89-3, symbol Transistor_BJT:BCX51
- added Q? (x2): CSD17303Q5, Package_TO_SOT_SMD:TDSON-8-1, symbol Transistor_FET:CSD17303Q5
- added R?: 1K, symbol Device:R_Small
- added U?: 74AHC1G04, symbol 74xGxx:74AHC1G04
- C?: value C_Small -> 1n5
- C?: value C_Small -> 100n
- D?: value D_Small -> BAS32
- D?: value LED_Small -> RED
- L?: value L_Small -> 1u5
- R?: value R_Small -> 33K
- R?: value R_Small -> 6K
- R? (x2): value R_Small -> 10K
- R? (x2): value R_Small -> 1K
- R?: value R_Small -> 5R
- R?: value R_Small -> 2K7
- R?: value R_Small -> 47K
- R? (x2): value R_Small -> 56R
- R? (x2): value R_Small -> 10R
- R?: value R_Small -> DNP
- R?: value R_Small -> 4K7
- R?: value R_Small -> 330R
Connections:
- net GND: now also C?.2, Q?.1 (S), Q?.1 (S), Q?.2 (S), Q?.2 (S), Q?.3 (S), Q?.3 (S), U?.3 (GND)
- net TX: now also U?.2
- net at R?.1, R?.1: now also C?.1
- net at R?.2, R?.2, R?.2: now also Q?.5 (D)
- net at R?.1: now also Q?.1 (B), Q?.1 (B), Q?.2 (C)
- net at R?.2: now also Q?.3 (E) (x2)
- net at D?.2 (A): now also Q?.2 (C)
- net at D?.1 (K), R?.2: now also Q?.5 (D)
- net at R?.2: now also Q?.4 (G)
- new net: R?.1, U?.4
- new net: Q?.4 (G), R?.2
- new net +5C: U?.5 (VCC)
Other:
- moved on the sheet: R?
